File: project/cad/recovery-physical-candidate/16_TF_Voltage_Translation.kicad_sch (KiCad schematic)
At the start: 4 parts, among them U95 NVT4858HKZ TF HS50 CANDIDATE

Commit message: Add R3 conditional footprint coverage and rename root project notes
Assign source-reviewed candidate footprints to L22-L26 and R574 only.
Coverage: 155 assigned, 99 unassigned; 254 components and 1509 pin bindings remain unchanged, with R528 DNP preserved.
Fresh KiCad 9.0.2 ERC: zero errors/warnings. Isolated fixture DRC passes; clearance negative control rejects as expected. Native recheck performed against exact publication copy.
Preserve all 27 frozen engineering changes plus their manifest. Root project notes renamed to 哦READ.MD as requested; existing history preserved.
Remaining gates include whole-board six-layer layout/routing, inductor under-body restrictions, thermal/timing/DFM and process qualification. Not production-ready.
Source manifest SHA256: 73eaddc8f8b261d1affe5c2291bbb92fcdbe4e234e270a22b1858ac4e41e9310
Delta ZIP SHA256: d36811aa21ddf584d98c255819cdc970d9e53bf3a46e318d5d2ef92ffa9bfec3
Verified tree: 3933ae06afe6062c348d20e1531ec2e9b6245dd9
Parts:
- R574: footprint (none) -> CMK230_Recovery_Passive_Candidates:Vishay_CRCW0201_SourceLand_PROCESS_CANDIDATE
