File: project/cad/recovery-physical-candidate/06_eMMC_1.kicad_sch (KiCad schematic)
At the start: 1 part, among them U3 MTFC16GAPALBH-AAT 16GB CANDID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

Commit message: Add R4 conditional BGA identity and footprint coverage
Assign U1/U2/U3 candidate footprints: 743 physical lands, 158 assigned and 96 remaining references. Preserve all 254 components, 1509 pin bindings, values and population attributes.
Fresh KiCad 9.0.2 checks on exact public copy: zero ERC violations, zero isolated six-layer geometry-fixture DRC violations, and native 390/200/153 numbered-pad recount. Independent 30+17 review checks are retained.
Correct eMMC maximum-body/courtyard drawing and K230 orientation cue without changing inherited copper/mask/paste pad subtrees. No historical routing, vias or fanout imported.
38 changed/new files only; retain exact root notes filename 哦READ.MD and prior history.
Not production-ready: whole-board six-layer fit/routing, DDR/PDN, stack/process, assembly, thermal and timing qualification remain open.
Source manifest SHA256: 450519dc83316734587bd46b5425656dd6c5a6aadd23309b589068988f3e482b
Delta ZIP SHA256: b23e8c294b8049e75d1469cf6f7ed302a6c7fc6852634157337af6cfaa789193
Verified tree: b8a12983eb12ea8eee55e8f13c8bedc421d4290d
Parts:
- U3: footprint (none) -> CMK230_Recovery_BGA_Candidates:MTFC16GAPALBH_AAT_BH153_NSMD030_ENGINEERING_ONLY
