File: project/cad/recovery-physical-candidate/08_Clock_Reset_Boot.kicad_sch (KiCad schematic)
At the start: 14 parts, among them Y1 32.768kHz / MPN TBD, Y2 X322524MOB4SI 24MHz CL12pF CA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

Commit message: Add R6 conditional passive footprint coverage
Assign candidates to 25 ordinary bias resistors and L21 only. Preserve all 254 component values, 457 nets, 1509 bindings and population attributes; R45/R47/R528 remain DNP. Coverage: 192 assigned, 62 gaps.
Exact publication-copy KiCad 9.0.2 export/ERC and full-component/graph comparison pass. L21 isolated six-layer fixture DRC passes; deliberate 1.40mm clearance rejects the 1.39mm gap. Native pad1 +X start mapping and recorded paste SVG aperture parity verified.
Keep independent graph, geometry and paste-override evidence. Three original explanatory/native-CAM SVGs inspected; no vendor pages, PDFs or runtime files uploaded.
60 changed/new files only; retain root 哦READ.MD and prior history. Not a complete core PCB or manufacturing, thermal, timing, switching-loop or DDR/PDN qualification.
Source manifest SHA256: 41e156fc71d4b10e1309578cfc231c354b290f847fc957d7bd48313e88f86145
Delta ZIP SHA256: 991fa45e6b49d84bdb60604ca1e232ea41bbe56994e89768a0dd62f8eb94a651
Verified tree: 4e28dc45a69ddc32ee629ba6cfef3bdfb46547ff
Parts:
- R43, R44, R45, R46, R47: footprint (none) -> CMK230_Recovery_Passive_Candidates:Vishay_CRCW0201_SourceLand_PROCESS_CANDIDATE
