File: project/cad/recovery-physical-candidate/15_Hardware_Reset_Interlock.kicad_sch (KiCad schematic)
At the start: 17 parts, among them U89 TPS3808G01DRVR VIN GUARD, U90 TPS3808G01DRVR RESET DELAY, U91 74AUP1G17GW,125 HIGH_TEMP CAN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, U92 74AUP2G97GUX DUAL SCHMITT AND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, U93 74AUP1G06GW,125 HIGH_TEMP CAN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

Commit message: Add R6 conditional passive footprint coverage
Assign candidates to 25 ordinary bias resistors and L21 only. Preserve all 254 component values, 457 nets, 1509 bindings and population attributes; R45/R47/R528 remain DNP. Coverage: 192 assigned, 62 gaps.
Exact publication-copy KiCad 9.0.2 export/ERC and full-component/graph comparison pass. L21 isolated six-layer fixture DRC passes; deliberate 1.40mm clearance rejects the 1.39mm gap. Native pad1 +X start mapping and recorded paste SVG aperture parity verified.
Keep independent graph, geometry and paste-override evidence. Three original explanatory/native-CAM SVGs inspected; no vendor pages, PDFs or runtime files uploaded.
60 changed/new files only; retain root 哦READ.MD and prior history. Not a complete core PCB or manufacturing, thermal, timing, switching-loop or DDR/PDN qualification.
Source manifest SHA256: 41e156fc71d4b10e1309578cfc231c354b290f847fc957d7bd48313e88f86145
Delta ZIP SHA256: 991fa45e6b49d84bdb60604ca1e232ea41bbe56994e89768a0dd62f8eb94a651
Verified tree: 4e28dc45a69ddc32ee629ba6cfef3bdfb46547ff
Parts:
- R527, R529, R530: footprint (none) -> CMK230_Recovery_Passive_Candidates:Vishay_CRCW0201_SourceLand_PROCESS_CANDIDATE

Commit message: R7: add conditional link footprints and fabricated copper features
Add ten footprint bindings and exclude JP1/TP81/TP82 from BOM; preserve all 254 values, 457 nets, 1509 pin/function/type/net bindings, on-board and DNP states. Coverage 202 assigned / 52 gaps.

Fresh KiCad 9.0.2 ERC passes. Independent exact-copy schematic, geometry, population, placement and CAM controls pass. Ten-reference isolated fixture has zero rule violations and three expected unrouted shared-net connections. Default paste still contains R528's two apertures despite DNP; explicit assembly/stencil variant remains a release gate. No complete core PCB, routing or manufacturing qualification.

Preserve 65 normalized source files plus manifest, source provenance, original CAD diagnostic SVG/CAM and root 哦READ.MD. Vendor originals excluded. All 1148 remote blobs verified against the local tree.

Manifest SHA256: 0fe14d3bf459b0f8046275165c57a58a2ab81769786d3e2496db5d605bf713fb
Delta ZIP SHA256: 3dfadf28c33240d59e85ee2e4374008a39fd3f1e564a0044020792ffa0f05c6e (230613 bytes)
Tree: c48cd1f548a5cd3a0ce28359b19fb4a988aab953
Parts:
- R528: footprint (none) -> CMK230_Recovery_Passive_Candidates:Vishay_CRCW0201_SourceLand_PROCESS_CANDIDATE
