File: project/cad/recovery-physical-candidate/11_DDR_USB_MIPI_Bias.kicad_sch (KiCad schematic)
At the start: 24 parts

Commit message: Add R6 conditional passive footprint coverage
Assign candidates to 25 ordinary bias resistors and L21 only. Preserve all 254 component values, 457 nets, 1509 bindings and population attributes; R45/R47/R528 remain DNP. Coverage: 192 assigned, 62 gaps.
Exact publication-copy KiCad 9.0.2 export/ERC and full-component/graph comparison pass. L21 isolated six-layer fixture DRC passes; deliberate 1.40mm clearance rejects the 1.39mm gap. Native pad1 +X start mapping and recorded paste SVG aperture parity verified.
Keep independent graph, geometry and paste-override evidence. Three original explanatory/native-CAM SVGs inspected; no vendor pages, PDFs or runtime files uploaded.
60 changed/new files only; retain root 哦READ.MD and prior history. Not a complete core PCB or manufacturing, thermal, timing, switching-loop or DDR/PDN qualification.
Source manifest SHA256: 41e156fc71d4b10e1309578cfc231c354b290f847fc957d7bd48313e88f86145
Delta ZIP SHA256: 991fa45e6b49d84bdb60604ca1e232ea41bbe56994e89768a0dd62f8eb94a651
Verified tree: 4e28dc45a69ddc32ee629ba6cfef3bdfb46547ff
Parts:
- R573, R61, R62: footprint (none) -> CMK230_Recovery_Passive_Candidates:Vishay_CRCW0201_SourceLand_PROCESS_CANDIDATE

Commit message: R9: add conditional eMMC bypass footprint candidates
Assign C64/C65/C69/C70/C71/C72 footprints while preserving all 254 values, other component metadata, 457 nets, 1509 complete pin/node bindings, BOM and population states. Coverage 221 assigned / 33 gaps. Internal EMMC_VDDIM, VCCQ and VCC roles remain distinct.

Fresh exact-copy KiCad 9.0.2 ERC and isolated geometry DRC pass. Full schematic metadata, fresh exported components/libparts/nets, source land/body ranges and saved/native CAM dimensions verified. Seven independent negative controls reject, including native physical 0.10mm clearance against 0.20mm rule. All 52 frozen source files plus manifest preserved byte-identically; all 1277 remote file hashes/sizes/modes match local tree.

Micron Table13 nominal/effective interpretation and combined hot/bias/aging capacitance remain qualification gates. No inferred VDDIM voltage or nominal capacitance change. Mask/stencil/courtyard process, JLC MOQ1, complete module placement/routing and physical validation remain open. Prior R528 DNP stencil gate remains. Vendor originals and runtime files excluded; history and root 哦READ.MD retained.

Manifest SHA256: 440a04548c9d5646c039cc5653e1596b5822c84bbe1afd09b54a9dba967daa69
Delta ZIP SHA256: 52fbc0a31d2438fb1fde49aa71446786239e050a4be5b1f352e35d117dfb85da (145858 bytes)
Tree: 711107a7002f46a80a3a24d8854ac899f6d9304e
Parts:
- C64, C69, C71: footprint (none) -> CMK230_EMMC_Bypass_Candidates:Murata_GRM188R71A225_ReflowMid_SOURCE_CANDIDATE
- C65, C70, C72: footprint (none) -> CMK230_EMMC_Bypass_Candidates:Murata_GRM155R71C104_ReflowMid_SOURCE_CANDIDATE
