File: project/cad/recovery-physical-candidate/10_Six_Rail_Power.kicad_sch (KiCad schematic)
At the start: 85 parts, among them U21 TPS62827ADMQ, U22 TPS628640BYCGR, U23 TPS628640BYCGR, U24 TPS62826ADMQ, U25 TPS62825ADMQ, U26 TPS62826ADMQ

Commit message: Add R3 conditional footprint coverage and rename root project notes
Assign source-reviewed candidate footprints to L22-L26 and R574 only.
Coverage: 155 assigned, 99 unassigned; 254 components and 1509 pin bindings remain unchanged, with R528 DNP preserved.
Fresh KiCad 9.0.2 ERC: zero errors/warnings. Isolated fixture DRC passes; clearance negative control rejects as expected. Native recheck performed against exact publication copy.
Preserve all 27 frozen engineering changes plus their manifest. Root project notes renamed to 哦READ.MD as requested; existing history preserved.
Remaining gates include whole-board six-layer layout/routing, inductor under-body restrictions, thermal/timing/DFM and process qualification. Not production-ready.
Source manifest SHA256: 73eaddc8f8b261d1affe5c2291bbb92fcdbe4e234e270a22b1858ac4e41e9310
Delta ZIP SHA256: d36811aa21ddf584d98c255819cdc970d9e53bf3a46e318d5d2ef92ffa9bfec3
Verified tree: 3933ae06afe6062c348d20e1531ec2e9b6245dd9
Parts:
- L22, L23: footprint (none) -> CMK230_Inductor_Candidates:Murata_DFE201612E-R24M_P2_SOURCE_LAND_PROCESS_CANDIDATE
- L24, L25, L26: footprint (none) -> CMK230_Inductor_Candidates:Murata_DFE201610E-R47M_P2_SOURCE_LAND_PROCESS_CANDIDATE

Commit message: Add R6 conditional passive footprint coverage
Assign candidates to 25 ordinary bias resistors and L21 only. Preserve all 254 component values, 457 nets, 1509 bindings and population attributes; R45/R47/R528 remain DNP. Coverage: 192 assigned, 62 gaps.
Exact publication-copy KiCad 9.0.2 export/ERC and full-component/graph comparison pass. L21 isolated six-layer fixture DRC passes; deliberate 1.40mm clearance rejects the 1.39mm gap. Native pad1 +X start mapping and recorded paste SVG aperture parity verified.
Keep independent graph, geometry and paste-override evidence. Three original explanatory/native-CAM SVGs inspected; no vendor pages, PDFs or runtime files uploaded.
60 changed/new files only; retain root 哦READ.MD and prior history. Not a complete core PCB or manufacturing, thermal, timing, switching-loop or DDR/PDN qualification.
Source manifest SHA256: 41e156fc71d4b10e1309578cfc231c354b290f847fc957d7bd48313e88f86145
Delta ZIP SHA256: 991fa45e6b49d84bdb60604ca1e232ea41bbe56994e89768a0dd62f8eb94a651
Verified tree: 4e28dc45a69ddc32ee629ba6cfef3bdfb46547ff
Parts:
- L21: footprint (none) -> CMK230_Recovery_Inductor_Candidates:Coilcraft_XFL4015_StartPin1_RIGHT_SOURCE_CANDIDATE
- R203, R204, R216, R217, R218, R219: footprint (none) -> CMK230_Recovery_Passive_Candidates:Vishay_CRCW0201_SourceLand_PROCESS_CANDIDATE

Commit message: R7: add conditional link footprints and fabricated copper features
Add ten footprint bindings and exclude JP1/TP81/TP82 from BOM; preserve all 254 values, 457 nets, 1509 pin/function/type/net bindings, on-board and DNP states. Coverage 202 assigned / 52 gaps.

Fresh KiCad 9.0.2 ERC passes. Independent exact-copy schematic, geometry, population, placement and CAM controls pass. Ten-reference isolated fixture has zero rule violations and three expected unrouted shared-net connections. Default paste still contains R528's two apertures despite DNP; explicit assembly/stencil variant remains a release gate. No complete core PCB, routing or manufacturing qualification.

Preserve 65 normalized source files plus manifest, source provenance, original CAD diagnostic SVG/CAM and root 哦READ.MD. Vendor originals excluded. All 1148 remote blobs verified against the local tree.

Manifest SHA256: 0fe14d3bf459b0f8046275165c57a58a2ab81769786d3e2496db5d605bf713fb
Delta ZIP SHA256: 3dfadf28c33240d59e85ee2e4374008a39fd3f1e564a0044020792ffa0f05c6e (230613 bytes)
Tree: c48cd1f548a5cd3a0ce28359b19fb4a988aab953
Parts:
- R205, R206: footprint (none) -> CMK230_Passive_Candidates:Vishay_TNPW0402_IPC7351_SourceLand_PROCESS_CANDIDATE
- R220: footprint (none) -> CMK230_Recovery_Link_Candidates:Vishay_WSL0603_9_SourceLand_PROCESS_CANDIDATE
- R221: footprint (none) -> CMK230_Recovery_Passive_Candidates:Vishay_CRCW0201_SourceLand_PROCESS_CANDIDATE

Commit message: R8: add conditional ferrite and feedforward source lands
Add thirteen footprint assignments: FB202-FB210 and C202/C219/C224/C229. Preserve all other component attributes, 254 values, 457 nets, 1509 pin/function/type/net bindings and BOM/population flags. Coverage 215 assigned / 39 gaps.

Fresh exact-copy KiCad 9.0.2 ERC and isolated geometry DRC pass. Native save/reload and complete copper/mask/paste aperture geometry match source CAM. Eight independent negative controls reject as expected, including physical clearance violations. All 89 frozen public source files plus manifest are preserved byte-identically; 1231 remote file hashes, sizes and modes match the local tree. Vendor originals and runtime files excluded; root 哦READ.MD retained.

Murata 18/35/70um variants remain distinct; the bound 18um local reservation does not approve the six-layer copper stack. Nominal mask openings contain zero registration allowance. Hot DCR, DC-bias filtering, continuing copper, feedforward loop behavior and factory process remain open. Prior R528 DNP stencil gate remains. No complete core layout or production qualification.

Manifest SHA256: cb780c38a4bc46eb86edf4b3e3dca31259c11cac5051fe36df7911f823e3bc0a
Delta ZIP SHA256: c1d0c019ab6488d189437282ee14b54dc892c91dc699cdcbd9cfd330c265dded (218776 bytes)
Tree: 578e53278763a346f092c8abf719e7ba9fb38a0f
Parts:
- C202, C219, C224, C229: footprint (none) -> CMK230_Filter_Feedforward_Candidates:KEMET_C0402_C0G_DensityB_SOURCE_CANDIDATE
- FB202, FB203, FB204, FB205, FB206, FB207, FB208, FB209, FB210: footprint (none) -> CMK230_Filter_Feedforward_Candidates:Murata_BLM15PX121_18um_SourcePattern_CONDITIONAL

Commit message: R11: add nine conditional 22uF source-land assignments
Assign C206-C208, C212-C214, C540/C552/C562 to the Samsung CL31B226 source-land candidate. Preserve all 254 values and other non-footprint identities, 457 nets, 1509 complete pin bindings and DNP/BOM/on-board flags. Coverage 230 assigned / 24 gaps.

Exact-copy independent audit passes all 77 checks: source schematic/generator scope, library ownership, input/source hashes, geometry and native CAM. Fresh KiCad 9.0.2 ERC and isolated fixture DRC pass. Six negative controls reject, including a physical native clearance violation. Courtyard clearance is 0.25mm from the mask envelope to the inner edge of its 0.05mm stroke.

All 50 frozen source files plus manifest preserved byte-identically. All 1429 remote file hashes/sizes/modes match local tree. Source-review historical input remains hash-identified; restored build_review.py matches its nested manifest. Vendor originals/runtime excluded, history and root 哦READ.MD preserved.

47uF proposal remains unselected; input-bank revisions remain unapplied. Combined biased/hot/aged effective capacitance, PDN/stability, full-core placement/routing and assembly/production qualification remain open. Isolated six-layer fixture does not approve the factory stack.

Manifest SHA256: b3027f4e2d5e34c68f64aa953d5ffb51e1b2352974e2279192d5e2459b55069d
Delta ZIP SHA256: 3ac08ec29f92146a0a1e548a2f95f7a83d257c990057a321455c4cee2121c917 (151404 bytes)
Tree: 565dd62d5809c02b1542320fd29f69c4952a8e14
Parts:
- C206, C207, C208, C212, C213, C214: footprint (none) -> CMK230_Bulk22_Candidates:Samsung_CL31B226_1206_ReflowMid_SOURCE_CANDIDATE
