File: project/cad/recovery-physical-candidate/12_Local_Decoupling.kicad_sch (KiCad schematic)
At the start: 77 parts

Commit message: R11: add nine conditional 22uF source-land assignments
Assign C206-C208, C212-C214, C540/C552/C562 to the Samsung CL31B226 source-land candidate. Preserve all 254 values and other non-footprint identities, 457 nets, 1509 complete pin bindings and DNP/BOM/on-board flags. Coverage 230 assigned / 24 gaps.

Exact-copy independent audit passes all 77 checks: source schematic/generator scope, library ownership, input/source hashes, geometry and native CAM. Fresh KiCad 9.0.2 ERC and isolated fixture DRC pass. Six negative controls reject, including a physical native clearance violation. Courtyard clearance is 0.25mm from the mask envelope to the inner edge of its 0.05mm stroke.

All 50 frozen source files plus manifest preserved byte-identically. All 1429 remote file hashes/sizes/modes match local tree. Source-review historical input remains hash-identified; restored build_review.py matches its nested manifest. Vendor originals/runtime excluded, history and root 哦READ.MD preserved.

47uF proposal remains unselected; input-bank revisions remain unapplied. Combined biased/hot/aged effective capacitance, PDN/stability, full-core placement/routing and assembly/production qualification remain open. Isolated six-layer fixture does not approve the factory stack.

Manifest SHA256: b3027f4e2d5e34c68f64aa953d5ffb51e1b2352974e2279192d5e2459b55069d
Delta ZIP SHA256: 3ac08ec29f92146a0a1e548a2f95f7a83d257c990057a321455c4cee2121c917 (151404 bytes)
Tree: 565dd62d5809c02b1542320fd29f69c4952a8e14
Parts:
- C540, C552, C562: footprint (none) -> CMK230_Bulk22_Candidates:Samsung_CL31B226_1206_ReflowMid_SOURCE_CANDIDATE
